File: N XOR gate/N XOR gate.kicad_pcb (KiCad board)
At the start: 2 copper layers, 23 parts

Commit message: Not Complete
Parts:
- moved REF** 14.0 mm to (141.0, 129.5)
- moved REF** 14.0 mm to (135.9, 134.6)
- moved REF** 14.0 mm to (148.6, 129.5)
- moved NPN 14.0 mm to (149.9, 134.6)
- moved NPN 14.0 mm to (142.2, 134.6)
- moved REF** 14.0 mm to (138.4, 146.1)
- moved NPN 11.5 mm to (139.7, 114.3)
- moved REF** 11.5 mm to (130.8, 109.2)
- moved REF** 11.5 mm to (154.9, 109.2)
- moved REF** 11.5 mm to (162.6, 109.2)
- moved REF** 11.5 mm to (125.7, 114.3)
- moved NPN 11.5 mm to (156.2, 114.3)
- moved NPN 11.5 mm to (163.8, 114.3)
- moved NPN 11.5 mm to (132.1, 114.3)
- moved REF** 11.5 mm to (138.4, 109.2)
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Routing:
- net (no net): track 158.6 -> 173.9 mm

Commit message: Add files via upload
Parts:
- removed the NPN at (154.9, 92.7)
- removed the REF** at (153.7, 87.6)
- removed the REF** at (160.0, 92.7)
- added 10KΩ: R_Axial_DIN0309_L9.0mm_D3.2mm_P5.08mm_Vertical, Resistor_THT:R_Axial_DIN0309_L9.0mm_D3.2mm_P5.08mm_Vertical, F.Cu at (129.5, 62.2)
- added 10KΩ: R_Axial_DIN0309_L9.0mm_D3.2mm_P5.08mm_Vertical, Resistor_THT:R_Axial_DIN0309_L9.0mm_D3.2mm_P5.08mm_Vertical, F.Cu at (158.8, 97.8)
- added 10KΩ: R_Axial_DIN0309_L9.0mm_D3.2mm_P5.08mm_Vertical, Resistor_THT:R_Axial_DIN0309_L9.0mm_D3.2mm_P5.08mm_Vertical, F.Cu at (142.2, 97.8)
- added 10KΩ: R_Axial_DIN0309_L9.0mm_D3.2mm_P5.08mm_Vertical, Resistor_THT:R_Axial_DIN0309_L9.0mm_D3.2mm_P5.08mm_Vertical, F.Cu at (128.3, 115.6)
- added 10KΩ: R_Axial_DIN0309_L9.0mm_D3.2mm_P5.08mm_Vertical, Resistor_THT:R_Axial_DIN0309_L9.0mm_D3.2mm_P5.08mm_Vertical, F.Cu at (152.4, 62.2)
- added 615Ω: R_Axial_DIN0309_L9.0mm_D3.2mm_P5.08mm_Vertical, Resistor_THT:R_Axial_DIN0309_L9.0mm_D3.2mm_P5.08mm_Vertical, F.Cu at (134.6, 62.2)
- added 615Ω: R_Axial_DIN0309_L9.0mm_D3.2mm_P5.08mm_Vertical, Resistor_THT:R_Axial_DIN0309_L9.0mm_D3.2mm_P5.08mm_Vertical, F.Cu at (162.6, 97.8)
- added 615Ω: R_Axial_DIN0309_L9.0mm_D3.2mm_P5.08mm_Vertical, Resistor_THT:R_Axial_DIN0309_L9.0mm_D3.2mm_P5.08mm_Vertical, F.Cu at (147.3, 97.8)
- added 615Ω: R_Axial_DIN0309_L9.0mm_D3.2mm_P5.08mm_Vertical, Resistor_THT:R_Axial_DIN0309_L9.0mm_D3.2mm_P5.08mm_Vertical, F.Cu at (133.3, 115.6)
- added 615Ω: R_Axial_DIN0309_L9.0mm_D3.2mm_P5.08mm_Vertical, Resistor_THT:R_Axial_DIN0309_L9.0mm_D3.2mm_P5.08mm_Vertical, F.Cu at (157.5, 62.2)
- added A LED: LED_D5.0mm, LED_THT:LED_D5.0mm, F.Cu at (133.3, 73.7)
- added AND LED: LED_D5.0mm, LED_THT:LED_D5.0mm, F.Cu at (143.5, 109.2)
- added B LED: LED_D5.0mm, LED_THT:LED_D5.0mm, F.Cu at (156.2, 73.7)
- added NPN: TO-92, Package_TO_SOT_THT:TO-92, F.Cu at (141.0, 62.2)
- added NPN: TO-92, Package_TO_SOT_THT:TO-92, F.Cu at (163.8, 62.2)
- added NPN: TO-92, Package_TO_SOT_THT:TO-92, F.Cu at (163.8, 68.6)
- added NPN: TO-92, Package_TO_SOT_THT:TO-92, F.Cu at (141.0, 68.6)
- added NPN: TO-92, Package_TO_SOT_THT:TO-92, F.Cu at (167.6, 102.9)
- added NPN: TO-92, Package_TO_SOT_THT:TO-92, F.Cu at (167.6, 108.0)
- added NPN: TO-92, Package_TO_SOT_THT:TO-92, F.Cu at (153.7, 97.8)
- added NPN: TO-92, Package_TO_SOT_THT:TO-92, F.Cu at (153.7, 104.1)
- added NPN: TO-92, Package_TO_SOT_THT:TO-92, F.Cu at (139.7, 115.6)
- added NPN: TO-92, Package_TO_SOT_THT:TO-92, F.Cu at (139.7, 121.9)
- added OR LED: LED_D5.0mm, LED_THT:LED_D5.0mm, F.Cu at (160.0, 109.2)
- added XOR LED: LED_D5.0mm, LED_THT:LED_D5.0mm, F.Cu at (132.1, 127.0)
- Input Header: renamed from REF**
- Output Header: renamed from REF**
- moved NPN 47.5 mm to (154.9, 88.9), turned to 270 degrees
- moved NPN 47.1 mm to (161.3, 88.9), turned to 270 degrees
- moved REF** 47.0 mm to (151.1, 90.2)
- moved REF** 47.0 mm to (156.2, 85.1)
- moved REF** 46.6 mm to (162.6, 85.1)
- moved NPN 24.3 mm to (142.2, 90.2)
- moved REF** 24.3 mm to (128.3, 90.2)
- moved 10K 24.3 mm to (133.3, 85.1)
- moved 10K 24.3 mm to (141.0, 85.1)
- moved NPN 24.3 mm to (134.6, 90.2)
- moved Input Header 20.7 mm to (142.2, 54.6)
- moved 10K 15.2 mm to (129.5, 102.9)
- moved NPN 15.2 mm to (130.8, 108.0)
- moved Output Header 13.1 mm to (144.8, 134.6)
- moved REF** 12.5 mm to (144.8, 125.7), turned to 0 degrees
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- renumbered REF** to 10K, REF** to 4.7K
Routing:
- net (no net): track 173.9 -> 807.5 mm
Other:
- board text added: "5V+"
- board text added: "A"
- board text added: "B"
- board text added: "Gnd"
- board text added: "NXOR"
- board text added: "XOR"
